File: PrototypeBoard.kicad_pcb (KiCad board)
At the start: 2 copper layers, 176 x 62 mm, 729 parts, among them J1 Conn_01x01_Socket, J2 Conn_01x01_Socket, J3 Conn_01x01_Socket, J4 Conn_01x01_Socket, J5 Conn_01x01_Socket, J6 Conn_01x01_Socket, P1 SMDpad, P10 SMDpad, P100 SMDpad, P101 SMDpad, P102 SMDpad, P103 SMDpad, P104 SMDpad, P105 SMDpad, P106 SMDpad, P107 SMDpad, P108 SMDpad, P109 SMDpad, P11 SMDpad, P110 SMDpad, P111 SMDpad, P112 SMDpad, P113 SMDpad, P114 SMDpad, P115 SMDpad, P116 SMDpad, P117 SMDpad, P118 SMDpad, P119 SMDpad, P12 SMDpad, P120 SMDpad, P121 SMDpad, P122 SMDpad, P123 SMDpad, P124 SMDpad, P125 SMDpad, P126 SMDpad, P127 SMDpad, P128 SMDpad, P129 SMDpad, P13 SMDpad, P130 SMDpad, P131 SMDpad, P132 SMDpad, P133 SMDpad, P134 SMDpad, P135 SMDpad, P136 SMDpad, P137 SMDpad, P138 SMDpad, P139 SMDpad, P14 SMDpad, P140 SMDpad, P141 SMDpad, P142 SMDpad, P143 SMDpad, P144 SMDpad, P145 SMDpad, P146 SMDpad, P147 SMDpad, P148 SMDpad, P149 SMDpad, P15 SMDpad, P150 SMDpad, P151 SMDpad, P152 SMDpad, P153 SMDpad, P154 SMDpad, P155 SMDpad, P156 SMDpad, P157 SMDpad, P158 SMDpad, P159 SMDpad, P16 SMDpad, P160 SMDpad, P161 SMDpad, P162 SMDpad, P163 SMDpad, P164 SMDpad, P165 SMDpad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

Commit message: 3
Parts:
- removed the P69 at (254.9, 61.5)
- added P213: SMDpad, Library:SMDpad_4x2.5mm, B.Cu at (101.6, 84.2)
- added P214: SMDpad, Library:SMDpad_4x2.5mm, F.Cu at (110.5, 70.0)
- added P215: SMDpad, Library:SMDpad_4x2.5mm, F.Cu at (107.8, 50.5)
- added P216: SMDpad, Library:SMDpad_4x2.5mm, B.Cu at (109.6, 68.1)
- added P217: SMDpad, Library:SMDpad_4x2.5mm, B.Cu at (108.2, 83.2)
- added P218: SMDpad, Library:SMDpad_4x2.5mm, F.Cu at (103.1, 87.8)
- moved R119 117.9 mm to (108.2, 46.2)
- moved R118 112.4 mm to (114.4, 46.2)
- moved P177 112.2 mm to (103.5, 42.0)
- moved R114 111.9 mm to (108.2, 42.0), turned to 0 degrees
- moved P180 111.3 mm to (104.3, 48.0)
- moved R115 104.7 mm to (114.9, 41.9), turned to 0 degrees
- moved R117 99.8 mm to (119.9, 48.4)
- moved R116 99.4 mm to (120.0, 43.6), turned to -90 degrees
- moved P178 93.3 mm to (123.1, 45.3)
- moved P179 92.2 mm to (124.3, 48.1)
Routing:
- net VEE: track 172.7 -> 180.5 mm
- net Net-(R114-Pad2): track 0.00 -> 3.68 mm
- net Net-(R115-Pad2): track 0.00 -> 3.57 mm
- net Net-(R117-Pad2): track 0.00 -> 3.26 mm
- net Net-(P177-Pad1): track 0.00 -> 3.15 mm
- net Net-(P178-Pad1): track 0.00 -> 3.14 mm
- net Net-(P180-Pad1): track 0.00 -> 3.12 mm
- net Net-(R118-Pad2): track 0.00 -> 3.12 mm
- net Net-(P179-Pad1): track 0.00 -> 3.00 mm

Commit message: 3
Parts:
- removed the P58 at (181.9, 43.7)
- removed the P58 at (209.9, 43.7)
- removed the P59 at (181.9, 46.5)
- removed the P59 at (209.9, 46.5)
- removed the P60 at (210.1, 49.1)
- removed the P60 at (182.1, 49.1)
- removed the P61 at (234.3, 49.1)
- removed the P61 at (206.3, 49.1)
- removed the P62 at (234.3, 46.5)
- removed the P62 at (206.3, 46.5)
- removed the P63 at (234.3, 43.7)
- removed the P63 at (206.3, 43.7)
- removed the R41 at (186.4, 43.7)
- removed the R41 at (214.4, 43.7)
- removed the R42 at (186.4, 46.5)
- removed the R42 at (214.4, 46.5)
- removed R43 (x2), R44 (x2), R45 (x2), R46 (x2), R47 (x2), R48 (x2), R49 (x2), R50 (x2), R51 (x2), R52 (x2): R, Resistor_SMD:R_1206_3216Metric_Pad1.30x1.75mm_HandSolder
- added P219: SMDpad, Library:SMDpad_4x2.5mm, B.Cu at (188.3, 48.3)
- added P220: SMDpad, Library:SMDpad_4x2.5mm, B.Cu at (193.7, 50.5)
- added P221: SMDpad, Library:SMDpad_4x2.5mm, B.Cu at (188.1, 56.8)
- added P222: SMDpad, Library:SMDpad_4x2.5mm, B.Cu at (188.4, 52.9)
- added P223: SMDpad, Library:SMDpad_4x2.5mm, B.Cu at (179.6, 48.1)
- added P224: SMDpad, Library:SMDpad_4x2.5mm, B.Cu at (143.8, 69.6)
- added P225: SMDpad, Library:SMDpad_4x2.5mm, B.Cu at (161.4, 71.7)
- added P226: SMDpad, Library:SMDpad_4x2.5mm, B.Cu at (211.2, 69.7)
- added P227: SMDpad, Library:SMDpad_4x2.5mm, B.Cu at (188.8, 70.8)
- added P58: SMDpad, Library:SMDpad_2x1.2mm, B.Cu at (232.7, 41.6)
- added P58: SMDpad, Library:SMDpad_2x1.2mm, B.Cu at (209.7, 41.6)
- added P59: SMDpad, Library:SMDpad_4x2.5mm, B.Cu at (193.9, 45.3)
- added P59: SMDpad, Library:SMDpad_4x2.5mm, B.Cu at (216.9, 45.3)
- added P60: SMDpad, Library:SMDpad_4x2.5mm, B.Cu at (236.1, 48.9)
- added P60: SMDpad, Library:SMDpad_4x2.5mm, B.Cu at (213.1, 48.9)
- added P61: SMDpad, Library:SMDpad_4x2.5mm, B.Cu at (183.5, 43.0)
- added P62: SMDpad, Library:SMDpad_4x2.5mm, B.Cu at (188.3, 43.0)
- added P63: SMDpad, Library:SMDpad_4x2.5mm, B.Cu at (183.4, 48.4)
- added Q6: IPD50R3K0CE, Package_TO_SOT_SMD:TO-252-2, B.Cu at (201.4, 45.5)
- added Q6: IPD50R3K0CE, Package_TO_SOT_SMD:TO-252-2, B.Cu at (224.4, 45.5)
- added R41: R, Resistor_SMD:R_1206_3216Metric_Pad1.30x1.75mm_HandSolder, B.Cu at (212.6, 44.2)
- added R41: R, Resistor_SMD:R_1206_3216Metric_Pad1.30x1.75mm_HandSolder, B.Cu at (235.6, 44.2)
- added R42: R, Resistor_SMD:R_1206_3216Metric_Pad1.30x1.75mm_HandSolder, B.Cu at (209.4, 45.4)
- added R42: R, Resistor_SMD:R_1206_3216Metric_Pad1.30x1.75mm_HandSolder, B.Cu at (232.4, 45.4)
Routing:
- net Net-(Q6-S): track 0.00 -> 15.7 mm
- net Net-(Q6-G): track 0.00 -> 14.6 mm
- net Net-(Q6-D): track 0.00 -> 10.2 mm
- net Net-(P59-Pad1): track 5.83 -> 0.00 mm
- net Net-(P60-Pad1): track 5.57 -> 0.00 mm
- net Net-(P63-Pad1): track 5.03 -> 0.00 mm
- net Net-(P62-Pad1): track 4.77 -> 0.00 mm
- net Net-(P61-Pad1): track 4.77 -> 0.00 mm
- net Net-(R43-Pad2): track 4.72 -> 0.00 mm
- net Net-(R42-Pad2): track 4.72 -> 0.00 mm
- net Net-(R41-Pad2): track 4.72 -> 0.00 mm
- net Net-(R46-Pad2): track 4.47 -> 0.00 mm
- net Net-(R45-Pad2): track 4.47 -> 0.00 mm
- net Net-(R49-Pad2): track 4.21 -> 0.00 mm
- net Net-(R48-Pad2): track 4.21 -> 0.00 mm
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