File: PrototypeBoard.kicad_sch (KiCad schematic)
At the start: 18 parts, among them P1 SMDpad, P2 SMDpad, P3 SMDpad, P4 SMDpad, U1 LM358

Commit message: 2
Parts:
- added C10, C11, C5, C6, C7: C, Capacitor_SMD:C_0805_2012Metric_Pad1.18x1.45mm_HandSolder, symbol Device:C
- added C8, C9: C_Polarized, Capacitor_THT:CP_Radial_D10.0mm_P5.00mm, symbol Device:C_Polarized
- added D1, D10, D2, D3, D4, D5, D6, D7, D8, D9: SS24, Diode_SMD:D_SMA, symbol Diode:SS24
- added H1, H2, H3, H4, H5, H6, H7: MountingHole, MountingHole:MountingHole_3.2mm_M3, symbol Mechanical:MountingHole
- added J1, J2, J3, J4, J5, J6: Conn_01x01_Socket, Library:Hole_1.2mm, symbol Connector:Conn_01x01_Socket
- added P10, P100, P11, P12, P13, P14, P15, P16, P17, P18, P19, P20, P21, P213, P214, P215, P216, P217, P218, P22, P23, P24, P25, P26, P27, P28, P29, P30, P31, P32, P33, P34, P35, P48, P49, P5, P50, P51, P52, P6, P66, P7, P8, P81, P82, P83, P84, P85, P86, P87, P88, P89, P9, P90, P91, P92, P93, P94, P95, P96, P97, P98, P99: SMDpad, Library:SMDpad_4x2.5mm, symbol New_Library:SMDpad
- added P101, P102, P103, P104, P105, P106, P107, P108, P109, P110, P111, P112, P113, P114, P115, P116, P117, P118, P119, P120, P121, P122, P123, P124, P125, P126, P127, P128, P129, P130, P131, P132, P133, P134, P135, P136, P137, P138, P139, P140, P141, P142, P143, P144, P145, P146, P147, P148, P149, P150, P151, P152, P153, P154, P155, P156, P157, P158, P159, P160, P161, P162, P163, P164, P165, P166, P167, P168, P169, P170, P171, P172, P173, P174, P175, P176, P177, P178, P179, P180, P181, P182, P183, P184, P185, P186, P187, P188, P189, P190, P191, P192, P193, P194, P195, P196, P197, P198, P199, P200, P201, P202, P203, P204, P205, P206, P207, P208, P209, P210, P211, P212, P36, P37, P38, P39, P40, P41, P42, P43, P44, P45, P46, P47, P53, P54, P55, P56, P57, P58, P59, P60, P61, P62, P63, P64, P65, P67, P68, P69, P70, P71, P72, P73, P74, P75, P76, P77, P78, P79, P80: SMDpad, Library:SMDpad_2x1.2mm, symbol New_Library:SMDpad
- added Q1, Q2, Q4, Q5: MMBT2222A, Package_TO_SOT_SMD:SOT-23, symbol Transistor_BJT:MMBT2222A
- added Q3: IPD50R3K0CE, Package_TO_SOT_SMD:TO-252-2, symbol Transistor_FET:IPD50R3K0CE
- added R10, R100, R101, R102, R103, R104, R105, R106, R107, R108, R109, R11, R110, R111, R112, R113, R114, R115, R116, R117, R118, R119, R12, R120, R121, R122, R124, R125, R13, R14, R15, R16, R17, R18, R19, R20, R21, R22, R23, R24, R25, R26, R27, R28, R29, R30, R31, R32, R33, R34, R35, R36, R37, R38, R39, R40, R41, R42, R43, R44, R45, R46, R47, R48, R49, R50, R51, R52, R53, R54, R55, R56, R57, R58, R59, R60, R61, R62, R63, R64, R65, R66, R67, R68, R69, R70, R71, R72, R73, R74, R75, R76, R77, R78, R79, R80, R81, R82, R83, R84, R85, R86, R87, R88, R89, R90, R91, R92, R93, R94, R95, R96, R97, R98, R99: R, Resistor_SMD:R_1206_3216Metric_Pad1.30x1.75mm_HandSolder, symbol Device:R
- added U10, U11, U3, U5: LM317_SOT-223, Package_TO_SOT_SMD:SOT-223-3_TabPin2, symbol Regulator_Linear:LM317_SOT-223
- added U2, U6: PCA9306D, Package_SO:SO-8_3.9x4.9mm_P1.27mm, symbol Interface:PCA9306D
- added U4: AD7794, Package_SO:TSSOP-24_4.4x7.8mm_P0.65mm, symbol Analog_ADC:AD7794
- added U7, U8, U9: INA181, Package_TO_SOT_SMD:SOT-23-6, symbol Amplifier_Current:INA181
Connections:
- net GND: now also C5.2, C8.2, C9.1, P18.1, P217.1, P218.1, P48.1, P49.1, P50.1, P51.1, P52.1, P86.1, P89.1, P90.1, P91.1, P92.1, R54.2, R59.2, R78.1, R82.1
- net VCC: now also C8.1, P100.1, P16.1, P19.1, P20.1, P21.1, P215.1, P216.1, P22.1, P23.1, P87.1, P97.1, P98.1, P99.1, R77.1, R79.1
- net VEE: now also C9.2, P17.1, P213.1, P214.1, P93.1, P94.1, P95.1, P96.1
- net at C3.1, P3.1, R6.1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: now also R83.1
- net at C1.2, R2.2, R4.1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: now also R84.1; no longer P4.1, U1.1
- net at C4.1, R8.1, R9.1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: now also P24.1, P25.1, P26.1, P27.1, P28.1, P88.1
- net at U1.5 (+): now also C5.1, P31.1, R53.2, R54.1, R85.1
- net at U1.6 (-): now also C6.1, C7.1, R55.2, R56.1, R58.2, R59.1
- net at U1.7: now also P34.1, R85.2, R86.2
- new net: P176.1, R113.1
- new net: R113.2, U11.1 (ADJ)
- new net: R43.2, R46.1
- new net: R46.2, R49.1
- new net: D6.2 (A), P106.1
- new net: R121.2, R122.1
- new net: P182.1, R122.2
- new net: P38.1, U2.6 (SCL2)
- new net: P168.1, U9.2 (GND)
- new net: R94.2, R96.1
- new net: R105.1, R96.2
- new net: R73.2, R74.1
- new net: P128.1, R74.2
- new net: P158.1, U7.1
- new net: P153.1, U7.2 (GND)
- new net: P156.1, U7.3 (+)
- new net: P157.1, U7.4 (-)
- new net: P154.1, U7.5 (REF)
- new net: P155.1, U7.6 (V+)
- new net: P193.1, P194.1
- new net: R70.2, R71.1
- new net: P114.1, R71.2
- new net: P165.1, U9.3 (+)
- new net: P207.1, P208.1
- new net: P56.1, U4.17 (AIN4+/REFIN2+)
- new net: P129.1, R77.2, U3.3 (VI)
- new net: R15.2, R19.1, R29.2, R30.1, R62.1
- new net: R20.2, R24.1, R33.2, R34.1, R62.2
- new net: R41.2, R44.1
- new net: R44.2, R47.1
- new net: P138.1, U6.1 (GND)
- new net: D7.1 (K), P107.1
- new net: P209.1, P210.1
- new net: P150.1, R103.1
- new net: Q5.3 (C), R103.2
- new net: P199.1, P200.1
- new net: D1.2 (A), D2.1 (K)
- new net: D2.2 (A), P102.1
- new net: P164.1, U8.1
- new net: P132.1, R79.2, U5.3 (VI)
- new net: R47.2, R50.1
- new net: R95.2, R97.1
- new net: R97.2, R98.1
- new net: P191.1, P192.1
- new net: P147.1, R100.1
- new net: Q4.3 (C), R100.2
- new net: P127.1, R72.1
- new net: P29.1, R38.1
- new net: P140.1, U6.8 (EN)
- new net: R19.2, R23.1, R32.2, R33.1, R63.1
- new net: R16.2, R20.1, R30.2, R31.1, R61.2
- new net: P181.1, R120.1
- new net: P65.1, U4.21 (AVDD)
- new net: R17.2, R21.1, R31.2
- new net: R21.2, R25.1, R34.2
- new net: P4.1, R83.2, R84.2, U1.1
- new net: R105.2, R106.1
- new net: R106.2, R107.1
- new net: P30.1, R39.1
- new net: Q2.3 (C), R39.2
- new net: P111.1, R66.1
- new net: R66.2, R67.1
- new net: P45.1, U4.9 (AIN2+)
- new net: Q1.2 (E), R37.1
- new net: P15.1, R37.2
- new net: C11.2, R80.2, R81.1, U5.1 (ADJ)
- new net: C11.1, P133.1, R81.2, R82.2
- new net: D1.1 (K), P101.1
- new net: Q1.1 (B), R36.2
- new net: Q1.3 (C), R35.2
- new net: R49.2, R52.1
- new net: P61.1, R52.2
- new net: R111.1, U11.2 (VO)
- new net: P171.1, R111.2
- new net: R48.2, R51.1
- new net: P62.1, R51.2
- new net: J5.1 (Pin_1), J6.1 (Pin_1)
- new net: P33.1, R55.1
- new net: C10.1, P131.1, R76.2, R78.2
- new net: R115.2, R116.1
- new net: P178.1, R116.2
- new net: P53.1, U4.10 (AIN2-)
- new net: P134.1, R80.1, U5.2 (VO)
- new net: D4.2 (A), P104.1
- new net: P162.1, U8.2 (GND)
- new net: C7.2, R56.2, R57.2, R58.1, R86.1
- new net: P13.1, R36.1
- new net: P177.1, R114.1
- new net: P184.1, R125.2
- new net: P7.1, R12.1
- new net: R12.2, R16.1, R27.2, R28.1, R60.2
- new net: P8.1, R13.1
- new net: P40.1, U2.7 (VREF2)
- new net: P179.1, R117.1
- new net: R117.2, R118.1
- new net: R89.2, R90.1
- new net: R90.2, R95.1
- new net: Q5.1 (B), R102.2
- new net: Q5.2 (E), R104.1
- new net: P144.1, R98.2
- new net: D7.2 (A), D8.1 (K)
- new net: R11.2, R15.1, R26.2, R27.1, R61.1
- new net: P211.1, P212.1
- new net: R72.2, R73.1
- new net: P32.1, R53.1
- new net: P187.1, P188.1
- new net: P10.1, R24.2, R63.2
- new net: P75.1, U4.24 (DIN)
- new net: P183.1, R124.1
- new net: C6.2, R57.1
- new net: P137.1, U6.2 (VREF1)
- new net: P135.1, U6.3 (SCL1)
- new net: P136.1, U6.4 (SDA1)
- new net: P142.1, U6.5 (SDA2)
- new net: P141.1, U6.6 (SCL2)
- new net: P139.1, U6.7 (VREF2)
- new net: R10.2, R14.1, R26.1
- new net: R92.2, R93.1
- new net: R93.2, R94.1
- new net: P163.1, U8.5 (REF)
- new net: P35.1, R40.2
- new net: P5.1, R10.1
- new net: P70.1, U4.6 (AIN6-/P2)
- new net: Q3.1 (G), R64.2, R65.2
- new net: P66.1, Q3.2 (D)
- new net: P81.1, Q3.3 (S), R65.1
- new net: P130.1, R75.1, U3.2 (VO)
- new net: P9.1, R25.2
- new net: R120.2, R121.1
- new net: P14.1, R35.1
- new net: P11.1, R23.2
- new net: D10.1 (K), D9.2 (A)
- new net: D10.2 (A), P110.1
- new net: P76.1, U4.3 (~{CS})
- new net: P59.1, R42.1
- new net: P60.1, R43.1
- new net: P205.1, P206.1
- new net: R118.2, R119.1
- new net: P180.1, R119.2
- new net: J1.1 (Pin_1), J2.1 (Pin_1)
- new net: P113.1, R69.1
- new net: R69.2, R70.1
- new net: C10.2, R75.2, R76.1, U3.1 (ADJ)
- new net: P74.1, U4.19 (PSW)
- new net: R112.2, U11.3 (VI)
- new net: R14.2, R18.1, R29.1
- new net: R18.2, R22.1, R32.1
- new net: R13.2, R17.1, R28.2
- new net: Q2.1 (B), R38.2
- new net: Q2.2 (E), R40.1
- new net: P6.1, R11.1, R60.1
- new net: R88.2, R89.1
- new net: R124.2, R125.1
- new net: P77.1, U4.1 (SCLK)
- new net: P54.1, U4.11 (AIN3+)
- new net: P55.1, U4.12 (AIN3-)
- new net: P72.1, U4.13 (REFIN1+)
- new net: P73.1, U4.14 (REFIN1-)
- new net: P67.1, U4.15 (AIN5+/IOUT2)
- new net: P68.1, U4.16 (AIN5-/IOUT1)
- new net: P57.1, U4.18 (AIN4-/REFIN2-)
- new net: P79.1, U4.2 (CLK)
- new net: P80.1, U4.20 (GND)
- new net: P78.1, U4.22 (DVDD)
- new net: P71.1, U4.23 (DOUT/~{RDY})
- new net: P69.1, U4.5 (AIN6+/P1)
- new net: P47.1, U4.7 (AIN1+)
- new net: P46.1, U4.8 (AIN1-)
- new net: P161.1, U8.6 (V+)
- new net: P148.1, R99.1
- new net: P175.1, R110.1
- new net: P201.1, P202.1
- new net: R67.2, R68.1
- new net: R114.2, R115.1
- new net: P63.1, R50.2
- new net: P39.1, U2.8 (EN)
- new net: P173.1, R108.1
- new net: R45.2, R48.1
- new net: P195.1, P196.1
- new net: P112.1, R68.2
- new net: R42.2, R45.1
- new net: P44.1, U2.1 (GND)
- new net: P166.1, U9.4 (-)
- new net: J3.1 (Pin_1), J4.1 (Pin_1), P36.1
- new net: P41.1, U2.2 (VREF1)
- new net: P159.1, U8.3 (+)
- new net: D3.2 (A), D4.1 (K)
- new net: P167.1, U9.6 (V+)
- new net: D3.1 (K), P103.1
- new net: Q4.1 (B), R99.2
- new net: P143.1, R87.1
- new net: R87.2, R88.1
- new net: D8.2 (A), P108.1
- new net: P64.1, R64.1
- new net: P12.1, R22.2
- new net: P203.1, P204.1
- new net: R108.2, U10.3 (VI)
- new net: P185.1, P186.1
- new net: P170.1, U9.1
- new net: P169.1, U9.5 (REF)
- new net: D5.1 (K), P105.1
- new net: D5.2 (A), D6.1 (K)
- new net: P37.1, U2.5 (SDA2)
- new net: P145.1, R91.1
- new net: R91.2, R92.1
- new net: P151.1, R104.2
- new net: P160.1, U8.4 (-)
- new net: P146.1, R107.2
- new net: P197.1, P198.1
- new net: P172.1, R109.2
- new net: P43.1, U2.4 (SDA1)
- new net: P152.1, R102.1
- new net: P58.1, R41.1
- new net: D9.1 (K), P109.1
- new net: P189.1, P190.1
- new net: P174.1, R112.1
- new net: R109.1, U10.2 (VO)
- new net: P42.1, U2.3 (SCL1)
- new net: R110.2, U10.1 (ADJ)
- new net: Q4.2 (E), R101.1
- new net: P149.1, R101.2
Other:
- moved on the sheet: C4, R8, R9, U1B, U1C

Commit message: 3
Parts:
- removed R43, R44, R45, R46, R47, R48, R49, R50, R51, R52: R, Resistor_SMD:R_1206_3216Metric_Pad1.30x1.75mm_HandSolder, symbol Device:R
- added P219, P220, P221, P222, P223, P224, P225, P226, P227: SMDpad, Library:SMDpad_4x2.5mm, symbol New_Library:SMDpad
- added Q6: IPD50R3K0CE, Package_TO_SOT_SMD:TO-252-2, symbol Transistor_FET:IPD50R3K0CE
- P59, P60, P61, P62, P63: footprint Library:SMDpad_2x1.2mm -> Library:SMDpad_4x2.5mm
Connections:
- net GND: now also P224.1, P225.1, P226.1, P227.1
- net at R41.2: now also R42.2, Q6.1 (G)
- net at R42.1: now also P60.1, Q6.3 (S); no longer P59.1
- new net: P59.1, Q6.2 (D)
